Commit message: v1.5: Real Baja dimensions, segmented terrain, PD path follower

File: src/baja_cloud_sim/urdf/baja_vehicle.urdf (robot description, URDF)
Before this commit: robot baja_vehicle, 7 links, 6 joints
Links:
- link base_link: geometry visual box size=1.70 1.50 0.40
Joints:
- joint front_left_steering_joint: origin xyz=0.715 0.655 -0.178 -> xyz=0.715 0.600 -0.178
- joint front_left_wheel_joint: origin xyz=0 0.09 0 -> xyz=0 0.06 0
- joint front_right_steering_joint: origin xyz=0.715 -0.655 -0.178 -> xyz=0.715 -0.600 -0.178
- joint front_right_wheel_joint: origin xyz=0 -0.09 0 -> xyz=0 -0.06 0
- joint rear_left_wheel_joint: origin xyz=-0.715 0.745 -0.178 -> xyz=-0.715 0.650 -0.178
- joint rear_right_wheel_joint: origin xyz=-0.715 -0.745 -0.178 -> xyz=-0.715 -0.650 -0.178

Commit message: feat(v1.1): update vehicle parameters to match real Baja SAE specs
- Mass: 292kg → 220kg (base_link 196 + 4×5 wheels + 2×2 steering)
- Chassis (L×W×H): 2.80×1.34×0.34 → 2.072×1.523×0.35
- Front track width: 1.49m → 1.32m
- Rear track width: 1.49m → 1.281m
- Wheelbase: 1.43m (unchanged, already correct)
- Recalculated chassis/wheel inertia for new mass and dimensions
- Updated planner params (vehicle_length/width) and scenario metadata

Files: model.sdf, baja_vehicle.urdf, params.yaml, scenario_generator.py, scenario.json

File: src/baja_cloud_sim/urdf/baja_vehicle.urdf (robot description, URDF)
Before this commit: robot baja_vehicle, 7 links, 6 joints
Links:
- link base_link: geometry visual box size=2.072 1.523 0.35
Joints:
- joint front_left_steering_joint: origin xyz=0.715 0.655 -0.178 -> xyz=0.715 0.57 -0.178
- joint front_right_steering_joint: origin xyz=0.715 -0.655 -0.178 -> xyz=0.715 -0.57 -0.178
- joint rear_left_wheel_joint: origin xyz=-0.715 0.745 -0.178 -> xyz=-0.715 0.6405 -0.178
- joint rear_right_wheel_joint: origin xyz=-0.715 -0.745 -0.178 -> xyz=-0.715 -0.6405 -0.178

Commit message: v1.4-real_lqr: Phase 0-4 complete
Phase 0: simulation baseline — freewheel, accel smoothing, continuous derating
Phase 1: speed profile — C2 B-spline, curvature-aware v(s)
Phase 2: LQR 4x4 — DARE, feedforward, speed-adaptive lookahead, DP improvements
Phase 3: state machine — 3-level hysteresis, speed-adaptive R, steering LPF
Phase 4: engineering — module split (core/), PlannedTrajectory

Core split into: geometry, collision, terrain, track, planner,
speed_profile, controller, config

File: src/baja_cloud_sim/urdf/baja_vehicle.urdf (robot description, URDF)
Before this commit: robot baja_vehicle, 7 links, 6 joints
Links:
- link base_link: geometry visual box size=2.8 1.34 0.34
Joints:
- joint front_left_steering_joint: origin xyz=0.715 0.57 -0.178 -> xyz=0.715 0.655 -0.178
- joint front_right_steering_joint: origin xyz=0.715 -0.57 -0.178 -> xyz=0.715 -0.655 -0.178
- joint rear_left_wheel_joint: origin xyz=-0.715 0.6405 -0.178 -> xyz=-0.715 0.745 -0.178
- joint rear_right_wheel_joint: origin xyz=-0.715 -0.6405 -0.178 -> xyz=-0.715 -0.745 -0.178

Commit message: v2.3: EPS 执行器模型 + 速度自适应反馈软化 + 双向曲率前瞻 + 三档速度分级
- actuator_adapter_node: 新增 EPS 模型(15°/s 转速上限 + 1° 死区, eps_tau=0 依赖 Gazebo 物理响应), 新增 /metrics/cmd_steer 与 /metrics/eps_actual_steer 诊断话题
- controller.py: 新增速度自适应反馈软化 beta(v)=1/(1+alpha*(v-v_ref)), 高速弱化反馈防蛇形
- speed_profile.py: 曲率限幅改为双向前瞻/后视窗口(curvature_lookahead_m=3.0), 根除弯切直过早加速
- params.yaml: max_steer_rate 恢复 1.2(去双重限速), steer_lowpass_alpha 0.22→0.5, max_lateral_accel=1.2, 三档速度 2.5/3.5/4.5
- evaluator/plot: 记录 eps_steer_rad, time_*.png 叠加实际齿条角
- 新增 tools/verify_eps.py(EPS 验证脚本) 与 real_car_params_regulation.md(实车参数对照)
- README 补充 EPS 章节、beta(v)、双向前瞻、三档速度、版本历史 v2.3

EPS 仅仿真层生效, 实车用不同 launch 替换 actuator_adapter_node 即去除

File: src/baja_cloud_sim/urdf/baja_vehicle.urdf (robot description, URDF)
Before this commit: robot baja_vehicle, 7 links, 6 joints
Links:
- link front_left_wheel: geometry visual cylinder length=0.18 radius=0.279
- link front_right_wheel: geometry visual cylinder length=0.18 radius=0.279
- link rear_left_wheel: geometry visual cylinder length=0.18 radius=0.279
- link rear_right_wheel: geometry visual cylinder length=0.18 radius=0.279
